File: PCB/Blueboard-Kicad/Blueboard-Kicad.kicad_pcb (KiCad board)
At the start: 2 copper layers, 224 parts, among them J1 OLED, SW1 M1, SW10 SHIFT, SW100 NM5, SW101 NM2, SW102 *, SW103 NM9, SW104 NM6, SW105 NM3, SW106 ., SW107 -, SW108 +, SW109 RotaryEncoder_Switch, SW11 CTL, SW110 Enter, SW111 RotaryEncoder_Switch, SW12 1, SW13 Q, SW14 A, SW15 Z, SW16 WIN, SW17 F1, SW18 2, SW19 W, SW2 ESC, SW20 S, SW21 X, SW22 ALT, SW23 F2, SW24 3, SW25 E, SW26 D, SW27 C, SW28 F3, SW29 4, SW3 M2, SW30 R, SW31 F, SW32 V, SW33 F4, SW34 5, SW35 T, SW36 G, SW37 B, SW38 SPACE, SW39 6, SW4 M3, SW40 Y, SW41 H, SW42 N, SW43 7, SW44 U, SW45 J, SW46 M, SW47 F5, SW48 F6, SW49 8, SW5 M4, SW50 I, SW51 K, SW52 <, SW53 ALT, SW54 F7, SW55 9, SW56 O, SW57 L, SW58 >, SW59 WIN, SW6 M5, SW60 F8, SW61 0, SW62 P, SW63 ;, SW64 ?, SW65 Menu, SW66 +, SW67 -, SW68 {, SW69 @, SW7 TILDA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

Commit message: Started Adding the Diodes to the PCB
Parts:
- D1, D10, D100, D101, D102, D103, D104, D105, D106, D107, D108, D11, D110, D12, D13, D14, D15, D16, D17, D18, D19, D2, D20, D21, D22, D23, D24, D25, D26, D27, D28, D29, D3, D30, D31, D32, D33, D34, D35, D36, D37, D38, D39, D4, D40, D41, D42, D43, D44, D45, D46, D47, D48, D49, D5, D50, D51, D52, D53, D54, D55, D56, D57, D58, D59, D6, D60, D61, D62, D63, D64, D65, D66, D67, D68, D69, D7, D70, D71, D72, D73, D74, D75, D76, D77, D78, D79, D8, D80, D81, D82, D83, D84, D85, D86, D87, D88, D89, D9, D90, D91, D92, D93, D94, D95, D96, D97, D98, D99: moved to B.Cu
- SW72: footprint Keyboard:SW_Cherry_MX1A_1.00u_PCB -> Keyboard:SW_Cherry_MX1A_1.25u_PCB
- SW75: footprint Keyboard:SW_Cherry_MX1A_1.50u_PCB -> Keyboard:SW_Cherry_MX1A_1.00u_PCB
- moved D94 333.2 mm to (430.3, 95.5), turned to 180 degrees
- moved D17 331.0 mm to (99.3, 64.0), turned to 180 degrees
- moved D76 320.8 mm to (272.5, 64.5), turned to 180 degrees
- moved D95 320.3 mm to (430.3, 115.0), turned to 180 degrees
- moved D73 314.5 mm to (314.0, 64.5), turned to 180 degrees
- moved D54 307.0 mm to (225.3, 64.5), turned to 180 degrees
- moved D33 305.1 mm to (158.5, 64.5), turned to 180 degrees
- moved D18 304.4 mm to (102.3, 95.5), turned to 180 degrees
- moved D92 293.7 mm to (430.3, 134.5), turned to 180 degrees
- moved D74 291.6 mm to (326.5, 95.5), turned to 180 degrees
- moved D91 291.0 mm to (402.0, 115.0), turned to 180 degrees
- moved D28 289.9 mm to (138.8, 64.0), turned to 180 degrees
- moved D12 288.8 mm to (83.0, 95.5), turned to 180 degrees
- moved D2 288.1 mm to (63.3, 64.5), turned to 180 degrees
- moved D19 286.8 mm to (111.8, 115.0), turned to 180 degrees
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Connections:
- D1 pad 2: unconnected-(D1-A-Pad2) -> Net-(D1-A)
- D9 pad 2: unconnected-(D9-A-Pad2) -> Net-(D9-A)
- SW1 pad 2: unconnected-(SW1-Pad2) -> Net-(D1-A)
- SW9 pad 2: unconnected-(SW9-Pad2) -> Net-(D9-A)

Commit message: Made alot of changes to the PCB
Parts:
- added ?: , , F.Cu at (374.0, 125.0)
- added ?: , , F.Cu at (71.4, 165.9)
- added ?: , , F.Cu at (61.4, 51.9)
- added ?: , , F.Cu at (522.9, 74.4)
- added REF**: MountingHole_3.2mm_M3, MountingHole:MountingHole_3.2mm_M3, F.Cu at (534.9, 163.9)
- moved D107 401.1 mm to (514.9, 92.4)
- moved D108 385.1 mm to (514.9, 121.9)
- moved D102 372.9 mm to (495.9, 92.4)
- moved D110 365.5 mm to (515.4, 160.4)
- moved D103 363.2 mm to (495.9, 111.9)
- moved D89 362.2 mm to (428.7, 60.9)
- moved D104 353.8 mm to (495.7, 131.4)
- moved D105 344.7 mm to (495.4, 150.9)
- moved D90 340.1 mm to (428.7, 92.4)
- moved D106 336.3 mm to (495.4, 170.4)
- moved D83 329.9 mm to (408.9, 60.9)
- moved D101 319.0 mm to (475.9, 150.9)
- moved D80 308.7 mm to (389.7, 60.9)
- moved D84 308.0 mm to (409.2, 92.4)
- moved D86 299.5 mm to (409.4, 111.9)
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Routing:
- net C1: track 0.00 -> 680.1 mm, vias 0 -> 1
- net C2: track 0.00 -> 670.0 mm, vias 0 -> 1
- net C3: track 0.00 -> 649.3 mm, vias 0 -> 1
- net C4: track 0.00 -> 633.6 mm, vias 0 -> 1
- net C5: track 0.00 -> 587.1 mm, vias 0 -> 1
- net C6: track 0.00 -> 562.7 mm, vias 0 -> 1
- net C7: track 0.00 -> 559.8 mm, vias 0 -> 1
- net R1: track 0.00 -> 515.8 mm
- net R3: track 0.00 -> 515.7 mm
- net C8: track 0.00 -> 512.5 mm, vias 0 -> 1
- net R5: track 0.00 -> 505.1 mm
- net R6: track 0.00 -> 504.0 mm
- net R4: track 0.00 -> 498.7 mm
- net R2: track 0.00 -> 490.9 mm
- net C10: track 0.00 -> 480.2 mm, vias 0 -> 1
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Other:
- board outline added: 520.4 x 139.6 mm
- board text added: "Blueboard"
- board text added: "Designed By Lawrence E Darbyshire in the UK"
- board text added: "I2C + C9-16 + C20-23"
- board text added: "ROT + VCC + C19-C1"

Commit message: Finalized PCB
Parts:
- added ?: , , F.Cu at (370.0, 165.0)
- moved ? 50.7 mm to (370.0, 74.5)
- moved ? 24.2 mm to (70.0, 74.5)
- moved REF** 8.70 mm to (527.0, 167.5)
- moved ? 4.78 mm to (526.5, 77.5)
- moved ? 1.64 mm to (70.0, 165.0)
- moved D22 0.64 mm to (140.2, 170.5)
- moved D17 0.64 mm to (125.7, 61.5)
- moved D23 0.64 mm to (145.2, 61.5)
- moved D28 0.64 mm to (165.2, 61.5)
- moved SW6 0.60 mm to (59.5, 159.8)
Connections:
- SW109 pad MP: (no net) -> GND
- SW111 pad MP: (no net) -> GND
Routing:
- net GND: track 202.1 -> 210.9 mm
- net R2: track 490.9 -> 489.3 mm
- net R6: track 504.0 -> 504.5 mm
- net (no net): vias 1 -> 0
Other:
- board size 520.4 x 139.6 mm -> 520.5 x 139.6 mm

Commit message: Forgot to Commit PCB Changes
Parts:
- removed ? (x5): , 
- removed the REF** at (527.0, 167.5)
- added REF**: MountingHole_3.2mm_M3, MountingHole:MountingHole_3.2mm_M3, F.Cu at (47.5, 247.5)
- added REF**: MountingHole_3.2mm_M3, MountingHole:MountingHole_3.2mm_M3, F.Cu at (338.0, 248.0)
- added REF**: MountingHole_3.2mm_M3, MountingHole:MountingHole_3.2mm_M3, F.Cu at (47.5, 147.5)
- added REF**: MountingHole_3.2mm_M3, MountingHole:MountingHole_3.2mm_M3, F.Cu at (492.5, 240.0)
- added REF**: MountingHole_3.2mm_M3, MountingHole:MountingHole_3.2mm_M3, F.Cu at (338.5, 146.5)
- ROT2: renamed from SW109; footprint Rotary_Encoder:RotaryEncoder_Alps_EC11E-Switch_Vertical_H20mm_MountingHoles -> Keyboard:RotaryEncoder_Alps_EC11E-Switch_Vertical_H20mm_MountingHoles
- ROT3: renamed from SW111; footprint Rotary_Encoder:RotaryEncoder_Alps_EC11E-Switch_Vertical_H20mm_MountingHoles -> Keyboard:RotaryEncoder_Alps_EC11E-Switch_Vertical_H20mm_MountingHoles
- SW12: renamed from SW73; footprint Keyboard:SW_Cherry_MX1A_1.25u_PCB -> Keyboard:SW_Cherry_MX1A_1.00u_PCB
- SW52: renamed from SW72; footprint Keyboard:SW_Cherry_MX1A_1.25u_PCB -> Keyboard:SW_Cherry_MX1A_1.00u_PCB
- SW53: renamed from SW75; footprint Keyboard:SW_Cherry_MX1A_1.00u_PCB -> Keyboard:SW_Cherry_MX1A_1.50u_PCB
- moved ROT2 97.7 mm to (454.2, 135.0), turned to 180 degrees
- moved U1 94.1 mm to (489.5, 135.5)
- moved J1 88.5 mm to (437.9, 138.3)
- moved SW16 85.3 mm to (390.7, 127.3)
- moved SW38 85.3 mm to (471.6, 155.9)
- moved D89 85.3 mm to (392.0, 137.8)
- moved SW15 85.1 mm to (371.6, 127.3)
- moved D102 85.1 mm to (453.9, 166.4)
- moved SW37 85.1 mm to (452.6, 155.9)
- moved D107 85.1 mm to (473.0, 166.4)
- moved D83 85.0 mm to (372.9, 137.8)
- moved SW14 85.0 mm to (352.6, 127.3)
- moved D80 84.9 mm to (353.9, 137.8)
- moved SW36 84.9 mm to (433.6, 155.9)
- moved D103 84.7 mm to (453.9, 185.5)
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- renumbered SW2 to SW1, SW76 to SW10, SW38 to SW100, SW53 to SW101, SW59 to SW102, SW65 to SW103, SW71 to SW104, SW85 to SW105, SW87 to SW106, SW93 to SW107, SW96 to SW108, SW106 to SW109, SW77 to SW11, SW79 to SW13, SW80 to SW14, SW83 to SW15, SW89 to SW16, SW1 to SW17, SW7 to SW18, SW12 to SW19, SW17 to SW2, SW18 to SW20, SW24 to SW21, SW29 to SW22, SW34 to SW23, SW39 to SW24, SW43 to SW25, SW49 to SW26, SW55 to SW27, SW61 to SW28, SW67 to SW29, SW23 to SW3, SW66 to SW30, SW74 to SW31, SW81 to SW32, SW84 to SW33, SW90 to SW34, SW94 to SW35, SW98 to SW36, SW102 to SW37, SW107 to SW38, SW3 to SW39, SW28 to SW4, SW8 to SW40, SW13 to SW41, SW19 to SW42, SW25 to SW43, SW30 to SW44, SW35 to SW45, SW40 to SW46, SW44 to SW47, SW50 to SW48, SW56 to SW49, SW33 to SW5, SW62 to SW50, SW68 to SW51, SW82 to SW54, SW86 to SW55, SW91 to SW56, SW95 to SW57, SW99 to SW58, SW103 to SW59, SW47 to SW6, SW108 to SW60, SW4 to SW61, SW9 to SW62, SW14 to SW63, SW20 to SW64, SW26 to SW65, SW31 to SW66, SW36 to SW67, SW41 to SW68, SW45 to SW69, SW48 to SW7, SW51 to SW70, SW57 to SW71, SW63 to SW72, SW69 to SW73, SW78 to SW74, SW92 to SW75, SW100 to SW76, SW104 to SW77, SW5 to SW78, SW10 to SW79, SW54 to SW8, SW15 to SW80, SW21 to SW81, SW27 to SW82, SW32 to SW83, SW37 to SW84, SW42 to SW85, SW46 to SW86, SW52 to SW87, SW58 to SW88, SW64 to SW89, SW60 to SW9, SW70 to SW90, SW88 to SW91, SW97 to SW92, SW101 to SW93, SW105 to SW94, SW110 to SW95, SW6 to SW96, SW11 to SW97, SW16 to SW98, SW22 to SW99
Connections:
- ROT2 pad MP: GND -> (no net)
- ROT3 pad MP: GND -> (no net)
Routing:
- net GND: track 210.9 -> 360.4 mm, vias 0 -> 3
- net C23: track 221.6 -> 343.7 mm, vias 1 -> 3
- net C2: track 670.0 -> 561.0 mm, vias 1 -> 0
- net C1: track 680.1 -> 577.8 mm, vias 1 -> 0
- net C4: track 633.6 -> 532.2 mm, vias 1 -> 0
- net C3: track 649.3 -> 555.3 mm
- net C5: track 587.1 -> 493.2 mm, vias 1 -> 0
- net C22: track 246.4 -> 339.4 mm, vias 1 -> 3
- net C6: track 562.7 -> 473.6 mm, vias 1 -> 0
- net C7: track 559.8 -> 481.9 mm, vias 1 -> 0
- net C8: track 512.5 -> 447.1 mm
- net C21: track 244.0 -> 306.4 mm, vias 1 -> 3
- net R3: track 515.7 -> 465.9 mm
- net ENC1_SW: track 57.0 -> 9.66 mm, vias 1 -> 0
- net C18: track 379.2 -> 339.9 mm, vias 0 -> 2
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Other:
- board size 520.5 x 139.6 mm -> 490.5 x 138 mm
- board text added: "Designed By Lawri Darbyshire"
- board text added: "This Keyboard was Made for Blueprint & Finiancialy Funded By Hackclub x AMD"
- board text removed: "Designed By Lawrence E Darbyshire in the UK"
- board text removed: "I2C + C9-16 + C20-23"
- board text removed: "ROT + VCC + C19-C1"
